File: ICE40-Board.kicad_pcb (KiCad board)
At the start: 2 copper layers, 0 parts

Commit message: Starting routing
Parts:
- added 5V_H1: Conn_01x03, Connector_PinHeader_2.54mm:PinHeader_1x03_P2.54mm_Vertical, F.Cu at (62.2, 43.2)
- added CDONE_R1: R, Resistor_SMD:R_0603_1608Metric, F.Cu at (165.0, 69.8)
- added CLOCK1: SIT2001BI-S2-33E-25.000000G, SIT2001BC-S2-33E-25.0:SIT2001BC-S2-33E-25.0, F.Cu at (126.0, 45.2)
- added CLOCK_C1: 0.1uF, Capacitor_SMD:C_0603_1608Metric, F.Cu at (120.9, 37.8)
- added CONF_FLASH1: W25X20CLSNIG, W25X20CLSNIG:W25X20CLSNIG, F.Cu at (120.1, 69.6)
- added CONF_FLASH_C1: 0.1uF, Capacitor_SMD:C_0603_1608Metric, F.Cu at (119.4, 76.2)
- added DC_IN1: Barrel_Jack, Connector_BarrelJack:BarrelJack_Horizontal, F.Cu at (35.7, 35.9)
- added FLASH_H11: Conn_01x03, Connector_PinHeader_2.54mm:PinHeader_1x03_P2.54mm_Vertical, F.Cu at (107.4, 59.2)
- added FPGA_2V5_C1: 0.1uF, Capacitor_SMD:C_0603_1608Metric, F.Cu at (164.6, 81.3)
- added FPGA_C1: 1uF, Capacitor_SMD:C_0603_1608Metric, F.Cu at (150.6, 81.3)
- added FPGA_C10: 0.1uF, Capacitor_SMD:C_0603_1608Metric, F.Cu at (132.3, 54.4)
- added FPGA_C2: 0.1uF, Capacitor_SMD:C_0603_1608Metric, F.Cu at (145.0, 78.5)
- added FPGA_C3: 10nF, Capacitor_SMD:C_0603_1608Metric, F.Cu at (156.2, 79.2)
- added FPGA_C4: 1uF, Capacitor_SMD:C_0603_1608Metric, F.Cu at (165.9, 57.9)
- added FPGA_C5: 0.1uF, Capacitor_SMD:C_0603_1608Metric, F.Cu at (164.1, 75.7)
- added FPGA_C6: 10nF, Capacitor_SMD:C_0603_1608Metric, F.Cu at (166.6, 64.5)
- added FPGA_C7: 10uF, Capacitor_SMD:C_0603_1608Metric, F.Cu at (133.1, 75.7)
- added FPGA_C8: 0.1uF, Capacitor_SMD:C_0603_1608Metric, F.Cu at (133.1, 70.9)
- added FPGA_C9: 10uF, Capacitor_SMD:C_0603_1608Metric, F.Cu at (133.3, 59.4)
- added FPGA_VCCIO0_C1: 0.1uF, Capacitor_SMD:C_0603_1608Metric, F.Cu at (145.3, 85.1)
- added FPGA_VCCIO1_C1: 0.1uF, Capacitor_SMD:C_0603_1608Metric, F.Cu at (172.7, 74.4)
- added FPGA_VCCIO2_C1: 0.1uF, Capacitor_SMD:C_0603_1608Metric, F.Cu at (158.2, 86.1)
- added FPGA_VCCIO3_C1: 0.1uF, Capacitor_SMD:C_0603_1608Metric, F.Cu at (157.0, 46.7)
- added FPGA_VCC_SPI_C1: 0.1uF, Capacitor_SMD:C_0603_1608Metric, F.Cu at (171.2, 46.2)
- added FTDI1: FT4222HQ, Package_DFN_QFN:VQFN-32-1EP_5x5mm_P0.5mm_EP3.1x3.1mm, F.Cu at (71.4, 63.5)
- added FT_3V3_C1: 4.7uF, Capacitor_THT:CP_Radial_D5.0mm_P2.50mm, F.Cu at (64.1, 68.8)
- added FT_3V3_C2: 0.1uF, Capacitor_SMD:C_0603_1608Metric, F.Cu at (70.9, 75.2)
- added FT_C1: 27pF, Capacitor_SMD:C_0603_1608Metric, F.Cu at (81.5, 79.0)
- added FT_C2: 27pF, Capacitor_SMD:C_0603_1608Metric, F.Cu at (82.8, 83.8)
- added FT_C3: 27pF, Capacitor_SMD:C_0603_1608Metric, F.Cu at (80.3, 74.9)
- added FT_Crystal1: 12MHz, Crystal:Crystal_HC49-U_Vertical, F.Cu at (94.0, 72.0)
- added FT_R1: 1M, Resistor_SMD:R_0603_1608Metric, F.Cu at (80.3, 65.3)
- added FT_R2: 12k, Resistor_SMD:R_0603_1608Metric, F.Cu at (82.8, 61.2)
- added FT_R3: 47k, Resistor_SMD:R_0603_1608Metric, F.Cu at (76.5, 89.9)
- added FT_R4: 10k, Resistor_SMD:R_0603_1608Metric, F.Cu at (75.6, 75.2)
- added FT_R5: 1k, Resistor_SMD:R_0603_1608Metric, F.Cu at (75.9, 82.3)
- added FT_VCCIN_C1: 4.7uF, Capacitor_THT:CP_Radial_D5.0mm_P2.50mm, F.Cu at (64.1, 91.9)
- added FT_VCCIN_C2: 0.1uF, Capacitor_SMD:C_0603_1608Metric, F.Cu at (84.3, 70.9)
- added FT_VCCIO_C1: 4.7uF, Capacitor_THT:CP_Radial_D5.0mm_P2.50mm, F.Cu at (64.1, 80.8)
- added FT_VCCIO_C2: 0.1uF, Capacitor_SMD:C_0603_1608Metric, F.Cu at (163.1, 51.3)
- added IO_H1: Conn_02x13_Row_Letter_Last, Connector_PinHeader_2.54mm:PinHeader_2x13_P2.54mm_Vertical, F.Cu at (133.6, 98.0)
- added IO_H2: Conn_02x09_Row_Letter_Last, Connector_PinHeader_2.00mm:PinHeader_2x09_P2.00mm_Vertical, F.Cu at (187.2, 70.7)
- added IO_H3: Conn_02x13_Row_Letter_Last, Connector_PinHeader_2.54mm:PinHeader_2x13_P2.54mm_Vertical, F.Cu at (164.8, 33.0)
- added JP1: SCK, Jumper:SolderJumper-2_P1.3mm_Open_Pad1.0x1.5mm, F.Cu at (88.1, 36.1)
- added JP2: MOSI, Jumper:SolderJumper-2_P1.3mm_Open_Pad1.0x1.5mm, F.Cu at (87.9, 41.1)
- added JP3: MISO, Jumper:SolderJumper-2_P1.3mm_Open_Pad1.0x1.5mm, F.Cu at (87.7, 46.2)
- added JP4: SS, Jumper:SolderJumper-2_P1.3mm_Open_Pad1.0x1.5mm, F.Cu at (87.6, 50.8)
- added JP5: SolderJumper_2_Bridged, Jumper:SolderJumper-2_P1.3mm_Bridged_Pad1.0x1.5mm, F.Cu at (128.0, 81.5)
- added PLL_R1: 100, Resistor_SMD:R_0603_1608Metric, F.Cu at (132.8, 67.1)
- added PLL_R2: 100, Resistor_SMD:R_0603_1608Metric, F.Cu at (133.1, 63.5)
- added PROG_FLASH1: W25X20CLSNIG, W25X20CLSNIG:W25X20CLSNIG, F.Cu at (118.4, 57.4)
- added PROG_FLASH_C1: 0.1uF, Capacitor_SMD:C_0603_1608Metric, F.Cu at (118.1, 51.1)
- added Q1: 2N222, Package_TO_SOT_THT:TO-92_Inline, F.Cu at (146.6, 48.0)
- added REG1: ADP1712AUJZ-1.2, Package_TO_SOT_SMD:SOT-23-5, F.Cu at (109.5, 26.2)
- added REG1_C1: 2.2uF, Capacitor_SMD:C_0603_1608Metric, F.Cu at (107.7, 19.8)
- added REG1_C2: 10nF, Capacitor_SMD:C_0603_1608Metric, F.Cu at (117.6, 22.4)
- added REG1_C3: 2.2uF, Capacitor_SMD:C_0603_1608Metric, F.Cu at (121.9, 30.5)
- added REG2: ADP1712AUJZ-2.5, Package_TO_SOT_SMD:SOT-23-5, F.Cu at (80.3, 22.9)
- added REG2_C1: 2.2uF, Capacitor_SMD:C_0603_1608Metric, F.Cu at (88.6, 23.4)
- added REG2_C2: 10nF, Capacitor_SMD:C_0603_1608Metric, F.Cu at (76.5, 18.0)
- added REG2_C3: 2.2uF, Capacitor_SMD:C_0603_1608Metric, F.Cu at (83.8, 16.8)
- added REG3: ADP1712AUJZ-3.3, Package_TO_SOT_SMD:SOT-23-5, F.Cu at (57.4, 23.4)
- added REG3_C1: 2.2uF, Capacitor_SMD:C_0603_1608Metric, F.Cu at (48.5, 22.4)
- added REG3_C2: 10nF, Capacitor_SMD:C_0603_1608Metric, F.Cu at (56.9, 17.0)
- added REG3_C3: 2.2uF, Capacitor_SMD:C_0603_1608Metric, F.Cu at (47.5, 16.0)
- added RESET_R1: 10k, Resistor_SMD:R_0603_1608Metric, F.Cu at (132.8, 82.0)
- added SCK_R1: 10k, Resistor_SMD:R_0603_1608Metric, F.Cu at (109.4, 90.9)
- added SIT_R1: 1k, Resistor_SMD:R_0603_1608Metric, F.Cu at (119.1, 44.2)
- added SPI_H3: Conn_01x05, Connector_PinHeader_2.54mm:PinHeader_1x05_P2.54mm_Vertical, F.Cu at (97.8, 38.9)
- added SPI_R1: R, Resistor_SMD:R_0603_1608Metric, F.Cu at (100.8, 94.2)
- added SS_CONF_R1: 10k, Resistor_SMD:R_0603_1608Metric, F.Cu at (109.5, 95.8)
- added TP1: TestPoint, TestPoint:TestPoint_Pad_D1.5mm, F.Cu at (70.4, 118.9)
- added TP2: TestPoint, TestPoint:TestPoint_Pad_D1.5mm, F.Cu at (60.7, 118.9)
- added TP3: TestPoint, TestPoint:TestPoint_Pad_D1.5mm, F.Cu at (50.8, 118.9)
- added TP4: TestPoint, TestPoint:TestPoint_Pad_D1.5mm, F.Cu at (80.8, 118.9)
- added U1: ICE40HX4K-TQ144, Package_QFP:TQFP-144_20x20mm_P0.5mm, F.Cu at (149.6, 64.0)
- added USB1: USB_C_Receptacle_USB2.0, Connector_USB:USB_C_Receptacle_Palconn_UTC16-G, F.Cu at (33.4, 64.0)
- added USB_R1: 5.1k, Resistor_SMD:R_0603_1608Metric, F.Cu at (45.6, 62.6)
- added USB_R2: 100, Resistor_SMD:R_0603_1608Metric, F.Cu at (52.1, 62.6)
- added USB_R3: 5.1k, Resistor_SMD:R_0603_1608Metric, F.Cu at (45.5, 65.7)
- added USB_R4: 100, Resistor_SMD:R_0603_1608Metric, F.Cu at (51.9, 65.7)
- added USB_R5: 1M, Resistor_SMD:R_0603_1608Metric, F.Cu at (35.7, 72.3)
- added VBUS_C1: 4.7uF, Capacitor_THT:CP_Radial_D5.0mm_P2.50mm, F.Cu at (64.4, 57.7)
- added VBUS_C2: 0.1uF, Capacitor_SMD:C_0603_1608Metric, F.Cu at (40.0, 69.2)
- added VPP_H2: Conn_01x02, Connector_PinHeader_2.54mm:PinHeader_1x02_P2.54mm_Vertical, F.Cu at (74.9, 57.1)
Routing:
- net (no net): vias 0 -> 6
Other:
- copper layers 2 -> 4
